Commit message: finish gazebo

File: src/jaka_tracer_ocs2/resource/tracer_jaka/urdf/tracer_jaka_zu5.urdf (robot description, URDF)
Before this commit: robot tracer_jaka_zu5, 42 links, 41 joints
Links:
- link Link_0: geometry collision mesh filename=package://jaka_tracer_ocs2/resource/tracer_jaka/meshes/jaka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; visual mesh filename=package://jaka_tracer_ocs2/resource/tracer_jaka/meshes/jaka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
- link Link_1: geometry collision mesh filename=package://jaka_tracer_ocs2/resource/tracer_jaka/meshes/jaka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; visual mesh filename=package://jaka_tracer_ocs2/resource/tracer_jaka/meshes/jaka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
- link Link_2: geometry collision mesh filename=package://jaka_tracer_ocs2/resource/tracer_jaka/meshes/jaka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; visual mesh filename=package://jaka_tracer_ocs2/resource/tracer_jaka/meshes/jaka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
- link Link_3: geometry collision mesh filename=package://jaka_tracer_ocs2/resource/tracer_jaka/meshes/jaka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; visual mesh filename=package://jaka_tracer_ocs2/resource/tracer_jaka/meshes/jaka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
- link Link_4: geometry collision mesh filename=package://jaka_tracer_ocs2/resource/tracer_jaka/meshes/jaka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; visual mesh filename=package://jaka_tracer_ocs2/resource/tracer_jaka/meshes/jaka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
- link Link_5: geometry collision mesh filename=package://jaka_tracer_ocs2/resource/tracer_jaka/meshes/jaka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; visual mesh filename=package://jaka_tracer_ocs2/resource/tracer_jaka/meshes/jaka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
- link Link_6: geometry collision mesh filename=package://jaka_tracer_ocs2/resource/tracer_jaka/meshes/jaka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; visual mesh filename=package://jaka_tracer_ocs2/resource/tracer_jaka/meshes/jaka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
- link aluminium_2_base_link: geometry collision mesh filename=package://jaka_tracer_ocs2/resource/tracer_jaka/meshes/alum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; visual mesh filename=package://jaka_tracer_ocs2/resource/tracer_jaka/meshes/alum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
- link aluminium_3_base_link: geometry collision mesh filename=package://jaka_tracer_ocs2/resource/tracer_jaka/meshes/alum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; visual mesh filename=package://jaka_tracer_ocs2/resource/tracer_jaka/meshes/alum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
- link aluminium_4_base_link: geometry collision mesh filename=package://jaka_tracer_ocs2/resource/tracer_jaka/meshes/alum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; visual mesh filename=package://jaka_tracer_ocs2/resource/tracer_jaka/meshes/alum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
- link aluminium_base_link: geometry collision mesh filename=package://jaka_tracer_ocs2/resource/tracer_jaka/meshes/alum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; visual mesh filename=package://jaka_tracer_ocs2/resource/tracer_jaka/meshes/alum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
- link base_link: geometry collision mesh filename=package://jaka_tracer_ocs2/resource/tracer_jaka/meshes/trac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; visual mesh filename=package://jaka_tracer_ocs2/resource/tracer_jaka/meshes/trac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
- link camera_link: geometry collision box size=0.02505 0.09 0.025; visual mesh filename=package://jaka_tracer_ocs2/resource/tracer_jaka/meshes/real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
- link connector_base_link: geometry collision mesh filename=package://jaka_tracer_ocs2/resource/tracer_jaka/meshes/conn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; visual mesh filename=package://jaka_tracer_ocs2/resource/tracer_jaka/meshes/conn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
- link fl_castor_link: geometry collision cylinder length=0.002 radius=0.03724; visual mesh filename=package://jaka_tracer_ocs2/resource/tracer_jaka/meshes/trac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
- link fl_wheel_link: geometry collision mesh filename=package://jaka_tracer_ocs2/resource/tracer_jaka/meshes/trac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; visual mesh filename=package://jaka_tracer_ocs2/resource/tracer_jaka/meshes/trac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
- link fr_castor_link: geometry collision cylinder length=0.002 radius=0.03724; visual mesh filename=package://jaka_tracer_ocs2/resource/tracer_jaka/meshes/trac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
- link fr_wheel_link: geometry collision mesh filename=package://jaka_tracer_ocs2/resource/tracer_jaka/meshes/trac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; visual mesh filename=package://jaka_tracer_ocs2/resource/tracer_jaka/meshes/trac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
- link gripper_base_link: geometry collision mesh filename=package://jaka_tracer_ocs2/resource/tracer_jaka/meshes/dh_r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 scale=0.001 0.001 0.001; visual mesh filename=package://jaka_tracer_ocs2/resource/tracer_jaka/meshes/dh_r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 scale=0.001 0.001 0.001
- link gripper_finger1_finger_link: geometry collision mesh filename=package://jaka_tracer_ocs2/resource/tracer_jaka/meshes/dh_r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 scale=0.001 0.001 0.001; visual mesh filename=package://jaka_tracer_ocs2/resource/tracer_jaka/meshes/dh_r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 scale=0.001 0.001 0.001
- link gripper_finger1_finger_tip_link: geometry collision mesh filename=package://jaka_tracer_ocs2/resource/tracer_jaka/meshes/dh_r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 scale=0.001 0.001 0.001; visual mesh filename=package://jaka_tracer_ocs2/resource/tracer_jaka/meshes/dh_r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 scale=0.001 0.001 0.001
- link gripper_finger1_inner_knuckle_link: geometry collision mesh filename=package://jaka_tracer_ocs2/resource/tracer_jaka/meshes/dh_r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 scale=0.001 0.001 0.001; visual mesh filename=package://jaka_tracer_ocs2/resource/tracer_jaka/meshes/dh_r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 scale=0.001 0.001 0.001
- link gripper_finger1_knuckle_link: geometry collision mesh filename=package://jaka_tracer_ocs2/resource/tracer_jaka/meshes/dh_r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 scale=0.001 0.001 0.001; visual mesh filename=package://jaka_tracer_ocs2/resource/tracer_jaka/meshes/dh_r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 scale=0.001 0.001 0.001
- link gripper_finger2_finger_link: geometry collision mesh filename=package://jaka_tracer_ocs2/resource/tracer_jaka/meshes/dh_r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 scale=0.001 0.001 0.001; visual mesh filename=package://jaka_tracer_ocs2/resource/tracer_jaka/meshes/dh_r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 scale=0.001 0.001 0.001
- link gripper_finger2_finger_tip_link: geometry collision mesh filename=package://jaka_tracer_ocs2/resource/tracer_jaka/meshes/dh_r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 scale=0.001 0.001 0.001; visual mesh filename=package://jaka_tracer_ocs2/resource/tracer_jaka/meshes/dh_r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 scale=0.001 0.001 0.001
- link gripper_finger2_inner_knuckle_link: geometry collision mesh filename=package://jaka_tracer_ocs2/resource/tracer_jaka/meshes/dh_r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 scale=0.001 0.001 0.001; visual mesh filename=package://jaka_tracer_ocs2/resource/tracer_jaka/meshes/dh_r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 scale=0.001 0.001 0.001
- link gripper_finger2_knuckle_link: geometry collision mesh filename=package://jaka_tracer_ocs2/resource/tracer_jaka/meshes/dh_r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 scale=0.001 0.001 0.001; visual mesh filename=package://jaka_tracer_ocs2/resource/tracer_jaka/meshes/dh_r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 scale=0.001 0.001 0.001
- link jk_se_vi_200_link: geometry collision mesh filename=package://jaka_tracer_ocs2/resource/tracer_jaka/meshes/jk_s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 scale=0.001 0.001 0.001; visual mesh filename=package://jaka_tracer_ocs2/resource/tracer_jaka/meshes/jk_s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 scale=0.001 0.001 0.001
- link left_wheel_link: geometry collision mesh filename=package://jaka_tracer_ocs2/resource/tracer_jaka/meshes/trac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; visual mesh filename=package://jaka_tracer_ocs2/resource/tracer_jaka/meshes/trac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
- link right_wheel_link: geometry collision mesh filename=package://jaka_tracer_ocs2/resource/tracer_jaka/meshes/trac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; visual mesh filename=package://jaka_tracer_ocs2/resource/tracer_jaka/meshes/trac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
- link rl_castor_link: geometry collision cylinder length=0.002 radius=0.03724; visual mesh filename=package://jaka_tracer_ocs2/resource/tracer_jaka/meshes/trac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
- link rl_wheel_link: geometry collision mesh filename=package://jaka_tracer_ocs2/resource/tracer_jaka/meshes/trac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; visual mesh filename=package://jaka_tracer_ocs2/resource/tracer_jaka/meshes/trac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
- link rr_castor_link: geometry collision cylinder length=0.002 radius=0.03724; visual mesh filename=package://jaka_tracer_ocs2/resource/tracer_jaka/meshes/trac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
- link rr_wheel_link: geometry collision mesh filename=package://jaka_tracer_ocs2/resource/tracer_jaka/meshes/trac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; visual mesh filename=package://jaka_tracer_ocs2/resource/tracer_jaka/meshes/trac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
- link urbase_base_link: geometry collision mesh filename=package://jaka_tracer_ocs2/resource/tracer_jaka/meshes/seco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; visual mesh filename=package://jaka_tracer_ocs2/resource/tracer_jaka/meshes/seco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

File: src/jaka_tracer_ocs2/resource/tracer_jaka/urdf/tracer_jaka_zu5_demo.urdf (robot description, URDF)
Before this commit: robot tracer_jaka_zu5, 42 links, 41 joints
Links:
- link Link_0: geometry collision cylinder length=0.2 radius=0.075; visual mesh filename=package://jaka_tracer_ocs2/resource/tracer_jaka/meshes/jaka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
- link Link_1: geometry collision cylinder length=0.25 radius=0.075; visual mesh filename=package://jaka_tracer_ocs2/resource/tracer_jaka/meshes/jaka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
- link Link_2: geometry collision cylinder length=0.15 radius=0.06; collision cylinder length=0.25 radius=0.075
- link Link_3: geometry collision cylinder length=0.15 radius=0.045; collision cylinder length=0.15 radius=0.055
- link Link_4: geometry collision cylinder length=0.20 radius=0.045; visual mesh filename=package://jaka_tracer_ocs2/resource/tracer_jaka/meshes/jaka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
- link Link_5: geometry collision cylinder length=0.12 radius=0.045; visual mesh filename=package://jaka_tracer_ocs2/resource/tracer_jaka/meshes/jaka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
- link Link_6: geometry collision cylinder length=0.05 radius=0.04; visual mesh filename=package://jaka_tracer_ocs2/resource/tracer_jaka/meshes/jaka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
- link aluminium_2_base_link: geometry collision box size=0.025 0.025 0.20; visual mesh filename=package://jaka_tracer_ocs2/resource/tracer_jaka/meshes/alum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
- link aluminium_3_base_link: geometry collision box size=0.025 0.025 0.20; visual mesh filename=package://jaka_tracer_ocs2/resource/tracer_jaka/meshes/alum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
- link aluminium_4_base_link: geometry collision box size=0.025 0.025 0.20; visual mesh filename=package://jaka_tracer_ocs2/resource/tracer_jaka/meshes/alum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
- link aluminium_base_link: geometry collision box size=0.025 0.025 0.20; visual mesh filename=package://jaka_tracer_ocs2/resource/tracer_jaka/meshes/alum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
- link base_link: geometry collision box size=0.58 0.58 0.18; visual mesh filename=package://jaka_tracer_ocs2/resource/tracer_jaka/meshes/trac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
- link camera_link: geometry collision box size=0.02505 0.09 0.025; visual mesh filename=package://jaka_tracer_ocs2/resource/tracer_jaka/meshes/real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
- link connector_base_link: geometry collision box size=0.04 0.04 0.07; visual mesh filename=package://jaka_tracer_ocs2/resource/tracer_jaka/meshes/conn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
- link fl_castor_link: geometry collision cylinder length=0.04 radius=0.035; visual mesh filename=package://jaka_tracer_ocs2/resource/tracer_jaka/meshes/trac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
- link fl_wheel_link: geometry collision sphere radius=0.04; visual mesh filename=package://jaka_tracer_ocs2/resource/tracer_jaka/meshes/trac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
- link fr_castor_link: geometry collision cylinder length=0.04 radius=0.035; visual mesh filename=package://jaka_tracer_ocs2/resource/tracer_jaka/meshes/trac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
- link fr_wheel_link: geometry collision sphere radius=0.04; visual mesh filename=package://jaka_tracer_ocs2/resource/tracer_jaka/meshes/trac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
- link gripper_base_link: geometry collision box size=0.075 0.045 0.10; visual mesh filename=package://jaka_tracer_ocs2/resource/tracer_jaka/meshes/dh_r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 scale=0.001 0.001 0.001
- link gripper_finger1_finger_link: geometry collision box size=0.025 0.012 0.04; visual mesh filename=package://jaka_tracer_ocs2/resource/tracer_jaka/meshes/dh_r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 scale=0.001 0.001 0.001
- link gripper_finger1_finger_tip_link: geometry collision box size=0.025 0.018 0.045; visual mesh filename=package://jaka_tracer_ocs2/resource/tracer_jaka/meshes/dh_r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 scale=0.001 0.001 0.001
- link gripper_finger1_inner_knuckle_link: geometry collision box size=0.055 0.018 0.025; visual mesh filename=package://jaka_tracer_ocs2/resource/tracer_jaka/meshes/dh_r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 scale=0.001 0.001 0.001
- link gripper_finger1_knuckle_link: geometry collision box size=0.04 0.015 0.025; visual mesh filename=package://jaka_tracer_ocs2/resource/tracer_jaka/meshes/dh_r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 scale=0.001 0.001 0.001
- link gripper_finger2_finger_link: geometry collision box size=0.025 0.012 0.04; visual mesh filename=package://jaka_tracer_ocs2/resource/tracer_jaka/meshes/dh_r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 scale=0.001 0.001 0.001
- link gripper_finger2_finger_tip_link: geometry collision box size=0.025 0.018 0.045; visual mesh filename=package://jaka_tracer_ocs2/resource/tracer_jaka/meshes/dh_r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 scale=0.001 0.001 0.001
- link gripper_finger2_inner_knuckle_link: geometry collision box size=0.055 0.018 0.025; visual mesh filename=package://jaka_tracer_ocs2/resource/tracer_jaka/meshes/dh_r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 scale=0.001 0.001 0.001
- link gripper_finger2_knuckle_link: geometry collision box size=0.04 0.015 0.025; visual mesh filename=package://jaka_tracer_ocs2/resource/tracer_jaka/meshes/dh_r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 scale=0.001 0.001 0.001
- link jk_se_vi_200_link: geometry collision box size=0.07 0.07 0.07; visual mesh filename=package://jaka_tracer_ocs2/resource/tracer_jaka/meshes/jk_s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 scale=0.001 0.001 0.001
- link left_wheel_link: geometry collision cylinder length=0.08 radius=0.085; visual mesh filename=package://jaka_tracer_ocs2/resource/tracer_jaka/meshes/trac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
- link right_wheel_link: geometry collision cylinder length=0.08 radius=0.085; visual mesh filename=package://jaka_tracer_ocs2/resource/tracer_jaka/meshes/trac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
- link rl_castor_link: geometry collision cylinder length=0.04 radius=0.035; visual mesh filename=package://jaka_tracer_ocs2/resource/tracer_jaka/meshes/trac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
- link rl_wheel_link: geometry collision sphere radius=0.04; visual mesh filename=package://jaka_tracer_ocs2/resource/tracer_jaka/meshes/trac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
- link rr_castor_link: geometry collision cylinder length=0.04 radius=0.035; visual mesh filename=package://jaka_tracer_ocs2/resource/tracer_jaka/meshes/trac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
- link rr_wheel_link: geometry collision sphere radius=0.04; visual mesh filename=package://jaka_tracer_ocs2/resource/tracer_jaka/meshes/trac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
- link urbase_base_link: geometry collision box size=0.6 0.4 0.04; visual mesh filename=package://jaka_tracer_ocs2/resource/tracer_jaka/meshes/seco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

File: src/tracer_jaka_moveit_config/config/tracer_jaka_zu5.ros2_control.xacro (robot description, xacro)
@@ -7,5 +7,6 @@
                 <!-- By default, set up controllers for simulation. This won't work on real hardware -->
                 <!-- <plugin>jaka_hardware_interface/JakaHardwareInterface</plugin> -->
-                <plugin>mock_components/GenericSystem</plugin>
+                <!-- <plugin>mock_components/GenericSystem</plugin> -->
+                <plugin>gz_ros2_control/GazeboSimSystem</plugin>
                 <param name="robot_ip">10.5.5.100</param>
                 <param name="local_ip">10.5.5.166</param>
@@ -76,4 +77,15 @@
               <state_interface name="torque.z"/>
             </sensor>
+                        <!-- mobile base wheels -->
+            <joint name="left_wheel">
+              <command_interface name="velocity"/>
+              <state_interface name="position"/>
+              <state_interface name="velocity"/>
+            </joint>
+            <joint name="right_wheel">
+              <command_interface name="velocity"/>
+              <state_interface name="position"/>
+              <state_interface name="velocity"/>
+            </joint>
         </ros2_control>
     </xacro:macro>
