Commit message: finish osc2 real

File: src/tracer_jaka_gazebo/urdf/tracer_jaka.ros2_control.xacro (robot description, xacro)
@@ -18,8 +18,26 @@
         <xacro:unless value="${sim_mode}">
           <!-- 实机硬件接口示意：替换为 Tracer + Jaka 的真实硬件接口 -->
-          <plugin>fake_components/GenericSystem</plugin>
+          <!-- <plugin>fake_components/GenericSystem</plugin> -->
+           <plugin>jaka_hardware_interface/JakaHardwareInterface</plugin>
+                           <param name="robot_ip">10.5.5.100</param>
+                <param name="local_ip">10.5.5.203</param>
+                <!-- 力传感器偏置 -->
+                <param name="ft_bias_fx">-9.80</param>
+                <param name="ft_bias_fy">-6.78</param>
+                <param name="ft_bias_fz">-6.00</param>
+                <param name="ft_bias_tx">0.54</param>
+                <param name="ft_bias_ty">-0.63</param>
+                <param name="ft_bias_tz">0.03</param>
+                <param name="r_t_s_x">0.0</param>
+                <param name="r_t_s_y">-0.05</param>
+                <param name="r_t_s_z">-0.226</param>
+                <!-- 死区 -->
+                <param name="ft_deadband_force">1.0</param>
+                <param name="ft_deadband_torque">0.00</param>
+                <!-- 滤波系数 -->
+                <param name="ft_filter_alpha">0.1</param>
         </xacro:unless>
       </hardware>
-      <!-- ============ 差速底盘：两个驱动轮（速度控制） ============ -->
+      <!-- ============ 差速底盘：两个驱动轮（速度控制） ============
       <joint name="left_wheel">
         <command_interface name="velocity">
@@ -37,5 +55,5 @@
         <state_interface name="position"/>
         <state_interface name="velocity"/>
-      </joint>
+      </joint> -->
       <!-- ============ 6 DOF 机械臂：position + velocity ============ -->
       <!-- 同时声明 position/velocity 两种 command_interface，方便切换不同控制器；
@@ -47,13 +65,8 @@
             <param name="max">${upper}</param>
           </command_interface>
-          <command_interface name="velocity">
-            <param name="min">-3.14</param>
-            <param name="max"> 3.14</param>
-          </command_interface>
           <state_interface name="position">
             <param name="initial_value">0.0</param>
           </state_interface>
           <state_interface name="velocity"/>
-          <state_interface name="effort"/>
         </joint>
       </xacro:macro>

File: src/tracer_jaka_ocs2/config/tracer_jaka.ros2_control.xacro (robot description, xacro)
@@ -77,15 +77,4 @@
               <state_interface name="torque.z"/>
             </sensor>
-                        <!-- mobile base wheels
-            <joint name="left_wheel">
-              <command_interface name="velocity"/>
-              <state_interface name="position"/>
-              <state_interface name="velocity"/>
-            </joint>
-            <joint name="right_wheel">
-              <command_interface name="velocity"/>
-              <state_interface name="position"/>
-              <state_interface name="velocity"/>
-            </joint> -->
         </ros2_control>
     </xacro:macro>

Commit message: fixed some real and sim files

File: src/tracer_jaka_gazebo/urdf/tracer_jaka.ros2_control.xacro (robot description, xacro)
@@ -20,5 +20,5 @@
           <!-- <plugin>fake_components/GenericSystem</plugin> -->
            <plugin>jaka_hardware_interface/JakaHardwareInterface</plugin>
-                           <param name="robot_ip">10.5.5.100</param>
+                <param name="robot_ip">10.5.5.100</param>
                 <param name="local_ip">10.5.5.203</param>
                 <!-- 力传感器偏置 -->
@@ -39,21 +39,22 @@
         </xacro:unless>
       </hardware>
-      <!-- ============ 差速底盘：两个驱动轮（速度控制） ============
-      <joint name="left_wheel">
-        <command_interface name="velocity">
-          <param name="min">-10.0</param>
-          <param name="max"> 10.0</param>
-        </command_interface>
-        <state_interface name="position"/>
-        <state_interface name="velocity"/>
-      </joint>
-      <joint name="right_wheel">
-        <command_interface name="velocity">
-          <param name="min">-10.0</param>
-          <param name="max"> 10.0</param>
-        </command_interface>
-        <state_interface name="position"/>
-        <state_interface name="velocity"/>
-      </joint> -->
+        <xacro:if value="${sim_mode}">
+          <joint name="left_wheel">
+            <command_interface name="velocity">
+              <param name="min">-10.0</param>
+              <param name="max"> 10.0</param>
+            </command_interface>
+            <state_interface name="position"/>
+            <state_interface name="velocity"/>
+          </joint>
+          <joint name="right_wheel">
+            <command_interface name="velocity">
+              <param name="min">-10.0</param>
+              <param name="max"> 10.0</param>
+            </command_interface>
+            <state_interface name="position"/>
+            <state_interface name="velocity"/>
+          </joint>
+        </xacro:if>
       <!-- ============ 6 DOF 机械臂：position + velocity ============ -->
       <!-- 同时声明 position/velocity 两种 command_interface，方便切换不同控制器；
@@ -77,4 +78,14 @@
       <xacro:arm_joint name="joint_5" lower="-6.28" upper="6.28"/>
       <xacro:arm_joint name="joint_6" lower="-6.28" upper="6.28"/>
+        <xacro:unless value="${sim_mode}">
+              <sensor name="tcp_fts_sensor">
+              <state_interface name="force.x"/>
+              <state_interface name="force.y"/>
+              <state_interface name="force.z"/>
+              <state_interface name="torque.x"/>
+              <state_interface name="torque.y"/>
+              <state_interface name="torque.z"/>
+          </sensor>
+        </xacro:unless>
     </ros2_control>
   </xacro:macro>

File: src/tracer_jaka_gazebo/urdf/tracer_jaka.urdf.xacro (robot description, xacro)
@@ -194,5 +194,5 @@
     </inertial>
     <visual>
-      <origin rpy="0 0 -1.57" xyz="0 0 0"/>
+      <origin rpy="0 0 0" xyz="0 0 0"/>
       <geometry>
         <mesh filename="package://tracer_jaka_gazebo/resources/second_base/meshes/urbase_base_link.STL"/>
@@ -206,5 +206,5 @@
   </link>
   <joint name="tracer_base" type="fixed">
-    <origin rpy="0 0 1.57" xyz="0 0 0.218"/>
+    <origin rpy="0 0 3.14" xyz="0 0 0.218"/>
     <parent link="base_link"/>
     <child  link="urbase_base_link"/>
@@ -221,5 +221,5 @@
     <parent link="base_link"/>
     <child  link="jaka_base_link"/>
-    <origin rpy="-0.02 0 0" xyz="0 0 0.221"/>
+    <origin rpy="0 0 -1.57" xyz="0 0 0.221"/>
   </joint>
   <link name="Link_0">
