Commit message: add tracer_jaka_ocs2

File: src/tracer_jaka_gazebo/urdf/tracer_jaka.urdf.xacro (robot description, xacro)
@@ -21,5 +21,5 @@
       <origin rpy="1.57 0 1.57" xyz="0 0 0"/>
       <geometry>
-        <mesh filename="package://jaka_tracer_ocs2/resource/tracer_jaka/meshes/tracer_description/meshes/tracer_base_link_no_wheel.dae"/>
+        <mesh filename="package://tracer_jaka_gazebo/resources/tracer_description/meshes/tracer_base_link_no_wheel.dae"/>
       </geometry>
     </visual>
@@ -60,5 +60,5 @@
       <origin rpy="0 0 0" xyz="0 0 0"/>
       <geometry>
-        <mesh filename="package://jaka_tracer_ocs2/resource/tracer_jaka/meshes/tracer_description/meshes/tracer_wheel.dae"/>
+        <mesh filename="package://tracer_jaka_gazebo/resources/tracer_description/meshes/tracer_wheel.dae"/>
       </geometry>
     </visual>
@@ -87,5 +87,5 @@
       <origin rpy="0 0 0" xyz="0 0 0"/>
       <geometry>
-        <mesh filename="package://jaka_tracer_ocs2/resource/tracer_jaka/meshes/tracer_description/meshes/tracer_wheel.dae"/>
+        <mesh filename="package://tracer_jaka_gazebo/resources/tracer_description/meshes/tracer_wheel.dae"/>
       </geometry>
     </visual>
@@ -115,5 +115,5 @@
       <visual>
         <geometry>
-          <mesh filename="package://jaka_tracer_ocs2/resource/tracer_jaka/meshes/tracer_description/meshes/castor_joint.dae"/>
+          <mesh filename="package://tracer_jaka_gazebo/resources/tracer_description/meshes/castor_joint.dae"/>
         </geometry>
       </visual>
@@ -136,5 +136,5 @@
       <visual>
         <geometry>
-          <mesh filename="package://jaka_tracer_ocs2/resource/tracer_jaka/meshes/tracer_description/meshes/castor.dae"/>
+          <mesh filename="package://tracer_jaka_gazebo/resources/tracer_description/meshes/castor.dae"/>
         </geometry>
       </visual>
@@ -166,5 +166,5 @@
         <origin rpy="0 0 0" xyz="0 0 0"/>
         <geometry>
-          <mesh filename="package://jaka_tracer_ocs2/resource/tracer_jaka/meshes/aluminium/meshes/aluminium_base_link.STL"/>
+          <mesh filename="package://tracer_jaka_gazebo/resources/aluminium/meshes/aluminium_base_link.STL"/>
         </geometry>
         <material name="white"><color rgba="0.898 0.917 0.929 1"/></material>
@@ -196,5 +196,5 @@
       <origin rpy="0 0 0" xyz="0 0 0"/>
       <geometry>
-        <mesh filename="package://jaka_tracer_ocs2/resource/tracer_jaka/meshes/second_base/meshes/urbase_base_link.STL"/>
+        <mesh filename="package://tracer_jaka_gazebo/resources/second_base/meshes/urbase_base_link.STL"/>
       </geometry>
       <material name="plate_white"><color rgba="1 1 1 1"/></material>
@@ -231,5 +231,5 @@
     <visual>
       <geometry>
-        <mesh filename="package://jaka_tracer_ocs2/resource/tracer_jaka/meshes/jaka_zu5_meshes/Link_0.STL"/>
+        <mesh filename="package://tracer_jaka_gazebo/resources/jaka_zu5_meshes/Link_0.STL"/>
       </geometry>
       <material name="silver"><color rgba="0.84706 0.84706 0.84706 1"/></material>
@@ -253,5 +253,5 @@
     <visual>
       <geometry>
-        <mesh filename="package://jaka_tracer_ocs2/resource/tracer_jaka/meshes/jaka_zu5_meshes/Link_1.STL"/>
+        <mesh filename="package://tracer_jaka_gazebo/resources/jaka_zu5_meshes/Link_1.STL"/>
       </geometry>
       <material name="silver"/>
@@ -271,5 +271,5 @@
       <origin rpy="0 0 0" xyz="0 0 0.14315"/>
       <geometry>
-        <mesh filename="package://jaka_tracer_ocs2/resource/tracer_jaka/meshes/jaka_zu5_meshes/Link_2.STL"/>
+        <mesh filename="package://tracer_jaka_gazebo/resources/jaka_zu5_meshes/Link_2.STL"/>
       </geometry>
       <material name="silver"/>
@@ -296,5 +296,5 @@
     <visual>
       <geometry>
-        <mesh filename="package://jaka_tracer_ocs2/resource/tracer_jaka/meshes/jaka_zu5_meshes/Link_3.STL"/>
+        <mesh filename="package://tracer_jaka_gazebo/resources/jaka_zu5_meshes/Link_3.STL"/>
       </geometry>
       <material name="silver"/>
@@ -322,5 +322,5 @@
     <visual>
       <geometry>
-        <mesh filename="package://jaka_tracer_ocs2/resource/tracer_jaka/meshes/jaka_zu5_meshes/Link_4.STL"/>
+        <mesh filename="package://tracer_jaka_gazebo/resources/jaka_zu5_meshes/Link_4.STL"/>
       </geometry>
       <material name="silver"/>
@@ -339,5 +339,5 @@
     <visual>
       <geometry>
-        <mesh filename="package://jaka_tracer_ocs2/resource/tracer_jaka/meshes/jaka_zu5_meshes/Link_5.STL"/>
+        <mesh filename="package://tracer_jaka_gazebo/resources/jaka_zu5_meshes/Link_5.STL"/>
       </geometry>
       <material name="silver"/>
@@ -356,5 +356,5 @@
     <visual>
       <geometry>
-        <mesh filename="package://jaka_tracer_ocs2/resource/tracer_jaka/meshes/jaka_zu5_meshes/Link_6.STL"/>
+        <mesh filename="package://tracer_jaka_gazebo/resources/jaka_zu5_meshes/Link_6.STL"/>
       </geometry>
       <material name="silver"/>
@@ -425,5 +425,5 @@
       <origin rpy="0 0 0" xyz="0 0 -0.0315"/>
       <geometry>
-        <mesh filename="package://jaka_tracer_ocs2/resource/tracer_jaka/meshes/jk_se_vi_200/meshes/jk_se_vi_200_link.stl" scale="0.001 0.001 0.001"/>
+        <mesh filename="package://tracer_jaka_gazebo/resources/jk_se_vi_200/meshes/jk_se_vi_200_link.stl" scale="0.001 0.001 0.001"/>
       </geometry>
     </visual>
@@ -447,5 +447,5 @@
     <visual>
       <geometry>
-        <mesh filename="package://jaka_tracer_ocs2/resource/tracer_jaka/meshes/dh_robotics_ag95_description/meshes/visual/dh_base_link.STL" scale="0.001 0.001 0.001"/>
+        <mesh filename="package://tracer_jaka_gazebo/resources/dh_robotics_ag95_description/meshes/visual/dh_base_link.STL" scale="0.001 0.001 0.001"/>
       </geometry>
       <material name="silver"/>

Commit message: fixed some urdf visiual bug

File: src/tracer_jaka_gazebo/urdf/tracer_jaka.urdf.xacro (robot description, xacro)
@@ -19,5 +19,5 @@
   <link name="base_link">
     <visual>
-      <origin rpy="1.57 0 1.57" xyz="0 0 0"/>
+      <origin rpy="1.57 0 0" xyz="0 0 0"/>
       <geometry>
         <mesh filename="package://tracer_jaka_gazebo/resources/tracer_description/meshes/tracer_base_link_no_wheel.dae"/>
@@ -194,5 +194,5 @@
     </inertial>
     <visual>
-      <origin rpy="0 0 0" xyz="0 0 0"/>
+      <origin rpy="0 0 -1.57" xyz="0 0 0"/>
       <geometry>
         <mesh filename="package://tracer_jaka_gazebo/resources/second_base/meshes/urbase_base_link.STL"/>

Commit message: add mujoco sim

File: src/tracer_jaka_gazebo/urdf/tracer_jaka.urdf.xacro (robot description, xacro)
@@ -201,5 +201,5 @@
     </visual>
     <collision>
-      <origin rpy="0 0 0" xyz="-0.08 0 -0.0025"/>
+      <origin rpy="0 0 0" xyz="0.0 0.04 -0.0025"/>
       <geometry><box size="0.6 0.4 0.04"/></geometry>
     </collision>
@@ -438,33 +438,40 @@
     <child  link="jk_se_vi_200_link"/>
   </joint>
-  <!-- 夹爪 base（其余指节作 fixed，不参与 OCS2 控制） -->
-  <link name="gripper_base_link">
-    <inertial>
-      <mass value="0.83416"/>
-      <origin xyz="0 0 0.05"/>
-      <inertia ixx="0.0013016" ixy="0" ixz="0" iyy="0.00049972" iyz="0" izz="0.001498"/>
-    </inertial>
-    <visual>
-      <geometry>
-        <mesh filename="package://tracer_jaka_gazebo/resources/dh_robotics_ag95_description/meshes/visual/dh_base_link.STL" scale="0.001 0.001 0.001"/>
-      </geometry>
-      <material name="silver"/>
-    </visual>
-    <collision>
-      <origin rpy="0 0 0" xyz="0 0 0.05"/>
-      <geometry><box size="0.075 0.045 0.10"/></geometry>
-    </collision>
-  </link>
-  <joint name="gripper_base_joint" type="fixed">
+  <link name="tool0_and_camera_link">
+    <inertial>
+      <origin rpy="0 0 0" xyz="0 0 0"/>
+      <mass value="0.7"/>
+      <inertia ixx="0.001" ixy="0" ixz="0"
+              iyy="0.001" iyz="0"
+              izz="0.001"/>
+    </inertial>
+    <visual>
+      <origin rpy="0 0 0" xyz="0 0 0"/>
+      <geometry>
+        <mesh filename="package://tracer_jaka_gazebo/resources/tool0.STL" scale="0.001 0.001 0.001"/>
+      </geometry>
+    </visual>
+    <collision>
+      <origin rpy="0 0 0" xyz="0 0 0.005"/>
+      <geometry><cylinder length="0.04" radius="0.04"/></geometry>
+    </collision>
+  </link>
+  <joint name="tool0_and_camera_link_joint" type="fixed">
+    <origin rpy="0 0 3.14" xyz="0 0 0.0"/>
     <parent link="jk_se_vi_200_link"/>
-    <child  link="gripper_base_link"/>
-    <origin rpy="0 0 -0.7853" xyz="0 0 0.005"/>
-  </joint>
-  <!-- TCP -->
-  <link name="gripper_center_link"/>
-  <joint name="gripper_center_joint" type="fixed">
-    <origin rpy="0 0 -0.785398" xyz="0 0 0.225"/>
-    <parent link="jk_se_vi_200_link"/>
-    <child  link="gripper_center_link"/>
+    <child  link="tool0_and_camera_link"/>
+  </joint>
+  <link name="d435i_link">
+    <visual>
+      <origin rpy="0 0 0" xyz="0 0 0"/>
+      <geometry>
+        <mesh filename="package://tracer_jaka_gazebo/resources/realsense_d435.stl" scale="0.001 0.001 0.001"/>
+      </geometry>
+    </visual>
+  </link>
+  <joint name="d435i_joint" type="fixed">
+    <origin rpy="0 0 3.14" xyz="0 -0.085 0.03"/>
+    <parent link="tool0_and_camera_link"/>
+    <child  link="d435i_link"/>
   </joint>
   <!-- ==================== ros2_control + Gazebo 插件 ==================== -->

File: src/tracer_jaka_moveit_config/config/tracer_jaka_zu5.ros2_control.xacro (robot description, xacro)
@@ -6,24 +6,5 @@
             <hardware>
                 <!-- By default, set up controllers for simulation. This won't work on real hardware -->
-                <plugin>jaka_hardware_interface/JakaHardwareInterface</plugin>
-                <!-- <plugin>mock_components/GenericSystem</plugin> -->
-                <!-- <plugin>gz_ros2_control/GazeboSimSystem</plugin> -->
-                <param name="robot_ip">10.5.5.100</param>
-                <param name="local_ip">10.5.5.203</param>
-                <!-- 力传感器偏置 -->
-                <param name="ft_bias_fx">-9.80</param>
-                <param name="ft_bias_fy">-6.78</param>
-                <param name="ft_bias_fz">-6.00</param>
-                <param name="ft_bias_tx">0.54</param>
-                <param name="ft_bias_ty">-0.63</param>
-                <param name="ft_bias_tz">0.03</param>
-                <param name="r_t_s_x">0.0</param>
-                <param name="r_t_s_y">-0.05</param>
-                <param name="r_t_s_z">-0.226</param>
-                <!-- 死区 -->
-                <param name="ft_deadband_force">1.0</param>
-                <param name="ft_deadband_torque">0.00</param>
-                <!-- 滤波系数 -->
-                <param name="ft_filter_alpha">0.1</param>
+                <plugin>mock_components/GenericSystem</plugin>
             </hardware>
             <joint name="joint_1">
@@ -69,23 +50,4 @@
                 <state_interface name="velocity"/>
             </joint>
-            <sensor name="tcp_fts_sensor">
-              <state_interface name="force.x"/>
-              <state_interface name="force.y"/>
-              <state_interface name="force.z"/>
-              <state_interface name="torque.x"/>
-              <state_interface name="torque.y"/>
-              <state_interface name="torque.z"/>
-            </sensor>
-                        <!-- mobile base wheels
-            <joint name="left_wheel">
-              <command_interface name="velocity"/>
-              <state_interface name="position"/>
-              <state_interface name="velocity"/>
-            </joint>
-            <joint name="right_wheel">
-              <command_interface name="velocity"/>
-              <state_interface name="position"/>
-              <state_interface name="velocity"/>
-            </joint> -->
         </ros2_control>
     </xacro:macro>

File: src/tracer_jaka_moveit_config/config/tracer_jaka_zu5.urdf.xacro (robot description, xacro)
@@ -3,7 +3,7 @@
     <xacro:arg name="initial_positions_file" default="initial_positions.yaml" />
     <!-- Import tracer_jaka_zu5 urdf file -->
-    <xacro:include filename="$(find jaka_description)/urdf/tracer_jaka_zu5.urdf" />
-    <!-- Import control_xacro -->
-    <xacro:include filename="tracer_jaka_zu5.ros2_control.xacro" />
-    <xacro:tracer_jaka_zu5_ros2_control name="FakeSystem" initial_positions_file="$(arg initial_positions_file)"/>
+    <xacro:include filename="$(find tracer_jaka_mujoco)/urdf/tracer_jaka_zu5.urdf" />
+    <!-- Import control_xacro
+    <xacro:include filename="tracer_jaka_zu5.ros2_control.xacro" /> -->
+    <!-- <xacro:tracer_jaka_zu5_ros2_control name="FakeSystem" initial_positions_file="$(arg initial_positions_file)"/> -->
 </robot>
