Commit message: finish tracer_jaka mujoco sim

File: src/tracer_jaka_mujoco/urdf/tracer_jaka_zu5.urdf (robot description, URDF)
Before this commit: robot tracer_jaka_zu5, 31 links, 30 joints
Joints:
- joint tool0_and_camera_link_joint: origin xyz=0 0 0 rpy=0 0 -2.3561945 -> xyz=0 0 0 rpy=0 0 -0.7853
