Commit message: finish sim to real

File: src/tracer_jaka_mujoco/urdf/tracer_jaka_zu5_real.urdf (robot description, URDF)
Before this commit: robot tracer_jaka_zu5, 31 links, 30 joints
Links:
- link Link_0: geometry collision cylinder length=0.15 radius=0.06; visual mesh filename=package://tracer_jaka_mujoco/urdf/meshes/Link_0.STL
- link Link_1: geometry collision cylinder length=0.15 radius=0.06; visual mesh filename=package://tracer_jaka_mujoco/urdf/meshes/Link_1.STL
- link Link_2: geometry collision cylinder length=0.29 radius=0.05; visual mesh filename=package://tracer_jaka_mujoco/urdf/meshes/Link_2.STL
- link Link_3: geometry collision cylinder length=0.1 radius=0.045; collision cylinder length=0.15 radius=0.055
- link Link_4: geometry collision cylinder length=0.1 radius=0.045; visual mesh filename=package://tracer_jaka_mujoco/urdf/meshes/Link_4.STL
- link Link_5: geometry collision cylinder length=0.17 radius=0.045; visual mesh filename=package://tracer_jaka_mujoco/urdf/meshes/Link_5.STL
- link Link_6: geometry visual mesh filename=package://tracer_jaka_mujoco/urdf/meshes/Link_6.STL
- link aluminium_2_base_link: geometry visual mesh filename=package://tracer_jaka_mujoco/urdf/meshes/aluminium_base_lin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
- link aluminium_3_base_link: geometry visual mesh filename=package://tracer_jaka_mujoco/urdf/meshes/aluminium_base_lin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
- link aluminium_4_base_link: geometry visual mesh filename=package://tracer_jaka_mujoco/urdf/meshes/aluminium_base_lin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
- link aluminium_base_link: geometry visual mesh filename=package://tracer_jaka_mujoco/urdf/meshes/aluminium_base_lin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
- link base_link: geometry visual mesh filename=package://tracer_jaka_mujoco/urdf/meshes/tracer_base_link_n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
- link d435i_link: geometry visual mesh filename=package://tracer_jaka_mujoco/urdf/meshes/realsense_d435.stl
- link fl_castor_link: geometry visual mesh filename=package://tracer_jaka_mujoco/urdf/meshes/castor_joint.dae
- link fl_wheel_link: geometry collision sphere radius=0.04; visual mesh filename=package://tracer_jaka_mujoco/urdf/meshes/castor.dae
- link fr_castor_link: geometry visual mesh filename=package://tracer_jaka_mujoco/urdf/meshes/castor_joint.dae
- link fr_wheel_link: geometry collision sphere radius=0.04; visual mesh filename=package://tracer_jaka_mujoco/urdf/meshes/castor.dae
- link jk_se_vi_200_link: geometry visual mesh filename=package://tracer_jaka_mujoco/urdf/meshes/jk_se_vi_200_link.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 scale=0.001 0.001 0.001
- link left_wheel_link: geometry collision cylinder length=0.08 radius=0.065; visual mesh filename=package://tracer_jaka_mujoco/urdf/meshes/tracer_wheel.dae
- link right_wheel_link: geometry collision cylinder length=0.08 radius=0.065; visual mesh filename=package://tracer_jaka_mujoco/urdf/meshes/tracer_wheel.dae
- link rl_castor_link: geometry visual mesh filename=package://tracer_jaka_mujoco/urdf/meshes/castor_joint.dae
- link rl_wheel_link: geometry collision sphere radius=0.04; visual mesh filename=package://tracer_jaka_mujoco/urdf/meshes/castor.dae
- link rr_castor_link: geometry visual mesh filename=package://tracer_jaka_mujoco/urdf/meshes/castor_joint.dae
- link rr_wheel_link: geometry collision sphere radius=0.04; visual mesh filename=package://tracer_jaka_mujoco/urdf/meshes/castor.dae
- link tool0_and_camera_link: geometry collision cylinder length=0.27 radius=0.08; visual mesh filename=package://tracer_jaka_mujoco/urdf/meshes/tool0.STL scale=0.001 0.001 0.001
- link urbase_base_link: geometry collision box size=0.6 0.4 0.04; visual mesh filename=package://tracer_jaka_mujoco/urdf/meshes/urbase_base_link.S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
