Commit message: switch forward command controller

File: src/tracer_jaka_moveit_config/config/tracer_jaka_zu5.ros2_control.xacro (robot description, xacro)
@@ -6,5 +6,23 @@
             <hardware>
                 <!-- By default, set up controllers for simulation. This won't work on real hardware -->
-                <plugin>mock_components/GenericSystem</plugin>
+                <plugin>jaka_hardware_interface/JakaHardwareInterface</plugin>
+                <!-- <plugin>mock_components/GenericSystem</plugin> -->
+                <param name="robot_ip">10.5.5.100</param>
+                <param name="local_ip">10.5.5.127</param>
+                <!-- 力传感器偏置 -->
+                <param name="ft_bias_fx">-7.79</param>
+                <param name="ft_bias_fy">-7.63</param>
+                <param name="ft_bias_fz">-0.21</param>
+                <param name="ft_bias_tx">0.74</param>
+                <param name="ft_bias_ty">-0.73</param>
+                <param name="ft_bias_tz">-0.02</param>
+                <param name="r_t_s_x">-0.0080</param>
+                <param name="r_t_s_y">-0.0157</param>
+                <param name="r_t_s_z">0.27</param>
+                <!-- 死区 -->
+                <param name="ft_deadband_force">0.0</param>
+                <param name="ft_deadband_torque">0.00</param>
+                <!-- 滤波系数 -->
+                <param name="ft_filter_alpha">0.0</param>
             </hardware>
             <joint name="joint_1">
@@ -50,4 +68,12 @@
                 <state_interface name="velocity"/>
             </joint>
+            <sensor name="tcp_fts_sensor">
+              <state_interface name="force.x"/>
+              <state_interface name="force.y"/>
+              <state_interface name="force.z"/>
+              <state_interface name="torque.x"/>
+              <state_interface name="torque.y"/>
+              <state_interface name="torque.z"/>
+            </sensor>
         </ros2_control>
     </xacro:macro>

File: src/tracer_jaka_moveit_config/config/tracer_jaka_zu5.urdf.xacro (robot description, xacro)
@@ -4,6 +4,6 @@
     <!-- Import tracer_jaka_zu5 urdf file -->
     <xacro:include filename="$(find tracer_jaka_mujoco)/urdf/tracer_jaka_zu5.urdf" />
-    <!-- Import control_xacro
-    <xacro:include filename="tracer_jaka_zu5.ros2_control.xacro" /> -->
-    <!-- <xacro:tracer_jaka_zu5_ros2_control name="FakeSystem" initial_positions_file="$(arg initial_positions_file)"/> -->
+    <!-- Import control_xacro -->
+    <xacro:include filename="tracer_jaka_zu5.ros2_control.xacro" />
+    <xacro:tracer_jaka_zu5_ros2_control name="FakeSystem" initial_positions_file="$(arg initial_positions_file)"/>
 </robot>

File: src/tracer_jaka_mujoco/urdf/tracer_jaka_zu5_real.urdf (robot description, URDF)
Before this commit: robot tracer_jaka_zu5, 31 links, 30 joints
Joints:
- joint base_to_jaka: origin xyz=0 0 0.221 rpy=0 0 -1.57 -> xyz=0 0 0.221 rpy=0 0 -1.5708
- joint left_wheel: type continuous -> fixed
- joint right_wheel: type continuous -> fixed
- joint tool0_and_camera_link_joint: origin xyz=0 0 0 rpy=0 0 -2.3561945 -> xyz=0 0 0 rpy=0 0 -0.785398
